File: kicad/majestouch_stm32.kicad_pcb (KiCad board)
At the start: 2 copper layers, 50 x 18 mm, 20 parts, among them J1 Filco 1-18, J2 Filco 19-36, J3 BOOT, J4 RESET, U1 STM32F072CBT6, U2 AP2112K-3.3, U3 USBLC6-2SC6

Commit message: KiCad 9: upgrade the project files, silkscreen v1.0
Schematic and board saved in KiCad 9.0.9. The library-mismatch
warnings are excluded (1 ERC, 20 DRC): the STM32 symbol was redrawn in
the KiCad 9 library and the footprints differ only in 3D models and
graphics, pads are identical. 3D model paths now point to the KiCad 9
.step models. Gerbers exported from v0.1 and from these files with
KiCad 9.0.9 have the same tracks, vias, pads and zone outline.

check.py uses pcbnew.EDA_UNITS_MM (renamed in KiCad 9), CI runs in
kicad/kicad:9.0.9, and the renders are regenerated.
Other:
- board text added: "STM32 v1.0"
- board text removed: "STM32 v0.1"
